Commit message: changed limits and forces of revolving joints

File: data/gripper/dummy_robot.urdf (robot description, URDF)
Before this commit: robot dummy_robot, 7 links, 6 joints
Joints:
- joint gripper_pitch: limit lower=-31.4 upper=31.4 effort=10000 velocity=3.14 -> lower=-3.14 upper=3.14 effort=10000 velocity=3.14
- joint gripper_roll: limit lower=-31.4 upper=31.4 effort=100000 velocity=3.14 -> lower=-3.14 upper=3.14 effort=10000 velocity=3.14
- joint gripper_yaw: limit lower=-31.4 upper=31.4 effort=10000 velocity=3.14 -> lower=-3.14 upper=3.14 effort=10000 velocity=3.14
