Commit message: comments, limits of z control joint

File: data/gripper/dummy_xyz_robot.urdf (robot description, URDF)
Before this commit: robot dummy_robot, 4 links, 3 joints
Joints:
- joint center_z: limit lower=-0.25 upper=1 effort=1000.0 velocity=0.2 -> lower=-0.5 upper=0.5 effort=1000.0 velocity=0.2

Commit message: added visualisation of the joints

File: data/gripper/dummy_xyz_robot.urdf (robot description, URDF)
Before this commit: robot dummy_xyz_robot, 4 links, 3 joints
Links:
- link base_link: geometry visual sphere radius=0.01
- link end_effector_link: geometry visual sphere radius=0.01
- link y_control: geometry visual sphere radius=0.01
- link z_control: geometry visual sphere radius=0.01
