Commit message: added support for wsg_32

File: burg_toolkit/gripper_module/assets/gripper/wsg_32/model.urdf (robot description, URDF)
Before this commit: robot wsg_32_description, 5 links, 4 joints
Joints:
- joint wsg_50_gripper_base_joint_gripper_left: limit lower=-0.028 upper=0 effort=0 velocity=0 -> lower=-0.028 upper=0 effort=20 velocity=0.2
- joint wsg_50_gripper_base_joint_gripper_right: axis 1 0 0 -> 0 0 1; limit lower=0 upper=0.028 effort=0 velocity=0 -> lower=0 upper=0.028 effort=20 velocity=0.2

Commit message: changed wsg32 STL to VHACD

File: burg_toolkit/gripper_module/assets/gripper/wsg_32/model.urdf (robot description, URDF)
Before this commit: robot wsg_32_description, 5 links, 4 joints
Links:
- link hand_link: geometry collision mesh filename=meshes/hand_link_vhacd.obj; visual mesh filename=meshes/hand_link_vhacd.obj
- link left_universal_finger_link: mass 0.001 -> 0.03; geometry collision mesh filename=meshes/universal_finger_vhacd.obj; visual mesh filename=meshes/universal_finger_vhacd.obj
- link right_universal_finger_link: mass 0.001 -> 0.03; geometry collision mesh filename=meshes/universal_finger_vhacd.obj; visual mesh filename=meshes/universal_finger_vhacd.obj
- link wsg_50_gripper_base_link_gripper_left: mass 3.41920163633724E-06 -> 0.03; geometry collision mesh filename=meshes/left_finger_link_vhacd.obj; visual mesh filename=meshes/left_finger_link_vhacd.obj
- link wsg_50_gripper_base_link_gripper_right: mass 3.41920163633724E-06 -> 0.03; geometry collision mesh filename=meshes/right_finger_link_vhacd.obj; visual mesh filename=meshes/right_finger_link_vhacd.obj
