Commit message: vhacd, aligned visual shapes with collision shapes

File: burg_toolkit/gripper_module/assets/gripper/robotiq_2f_85/model.urdf (robot description, URDF)
Before this commit: robot robotiq_arg2f_85_model, 11 links, 10 joints
Links:
- link left_inner_finger: geometry collision mesh filename=./meshes/robotiq_arg2f_85_inner_finger_vhacd.obj scale=0.001 0.001 0.001
- link left_inner_knuckle: geometry collision mesh filename=./meshes/robotiq_arg2f_85_inner_knuckle_vhacd.obj scale=0.001 0.001 0.001; visual mesh filename=./meshes/robotiq_arg2f_85_inner_knuckle_vhacd.obj scale=0.001 0.001 0.001
- link left_outer_finger: geometry collision mesh filename=./meshes/robotiq_arg2f_85_outer_finger_vhacd.obj scale=0.001 0.001 0.001
- link left_outer_knuckle: geometry collision mesh filename=./meshes/robotiq_arg2f_85_outer_knuckle_vhacd.obj scale=0.001 0.001 0.001
- link right_inner_finger: geometry collision mesh filename=./meshes/robotiq_arg2f_85_inner_finger_vhacd.obj scale=0.001 0.001 0.001; visual mesh filename=./meshes/robotiq_arg2f_85_inner_finger_vhacd.obj scale=0.001 0.001 0.001
- link right_inner_knuckle: geometry collision mesh filename=./meshes/robotiq_arg2f_85_inner_knuckle_vhacd.obj scale=0.001 0.001 0.001; visual mesh filename=./meshes/robotiq_arg2f_85_inner_knuckle_vhacd.obj scale=0.001 0.001 0.001
- link right_outer_finger: geometry collision mesh filename=./meshes/robotiq_arg2f_85_outer_finger_vhacd.obj scale=0.001 0.001 0.001; visual mesh filename=./meshes/robotiq_arg2f_85_outer_finger_vhacd.obj scale=0.001 0.001 0.001
- link right_outer_knuckle: geometry collision mesh filename=./meshes/robotiq_arg2f_85_outer_knuckle_vhacd.obj scale=0.001 0.001 0.001; visual mesh filename=./meshes/robotiq_arg2f_85_outer_knuckle_vhacd.obj scale=0.001 0.001 0.001
- link robotiq_arg2f_base_link: geometry collision mesh filename=./meshes/robotiq_arg2f_base_link.stl; visual mesh filename=./meshes/robotiq_arg2f_base_link.stl

Commit message: removed comments

File: burg_toolkit/gripper_module/assets/gripper/robotiq_2f_85/model.urdf (robot description, URDF)
Before this commit: robot robotiq_arg2f_85_model, 11 links, 10 joints
Links:
- link left_inner_finger: geometry collision mesh filename=./meshes/robotiq_arg2f_85_inner_finger_vhacd.obj scale=0.001 0.001 0.001; visual mesh filename=./meshes/robotiq_arg2f_85_inner_finger_vhacd.obj scale=0.001 0.001 0.001
- link left_outer_finger: geometry collision mesh filename=./meshes/robotiq_arg2f_85_outer_finger_vhacd.obj scale=0.001 0.001 0.001; visual mesh filename=./meshes/robotiq_arg2f_85_outer_finger_vhacd.obj scale=0.001 0.001 0.001
- link left_outer_knuckle: geometry collision mesh filename=./meshes/robotiq_arg2f_85_outer_knuckle_vhacd.obj scale=0.001 0.001 0.001; visual mesh filename=./meshes/robotiq_arg2f_85_outer_knuckle_vhacd.obj scale=0.001 0.001 0.001
