Commit message: vhacd of stl files

File: burg_toolkit/gripper_module/assets/gripper/rg2/model.urdf (robot description, URDF)
Before this commit: robot rg2, 7 links, 6 joints
Links:
- link left_finger: geometry collision mesh filename=meshes/left_finger_vhacd.obj scale=0.001 0.001 0.001
- link left_inner: geometry collision mesh filename=meshes/left_inner_vhacd.obj scale=0.001 0.001 0.001; visual mesh filename=meshes/left_inner_vhacd.obj scale=0.001 0.001 0.001
- link left_outer: geometry collision mesh filename=meshes/left_outer_vhacd.obj scale=0.001 0.001 0.001
- link palm: geometry collision mesh filename=meshes/palm_vhacd.obj scale=0.001 0.001 0.001; visual mesh filename=meshes/palm_vhacd.obj scale=0.001 0.001 0.001
- link right_finger: geometry collision mesh filename=meshes/right_finger_vhacd.obj scale=0.001 0.001 0.001; visual mesh filename=meshes/right_finger_vhacd.obj scale=0.001 0.001 0.001
- link right_inner: geometry collision mesh filename=meshes/right_inner_vhacd.obj scale=0.001 0.001 0.001; visual mesh filename=meshes/right_inner_vhacd.obj scale=0.001 0.001 0.001
- link right_outer: geometry collision mesh filename=meshes/right_outer_vhacd.obj scale=0.001 0.001 0.001; visual mesh filename=meshes/right_outer_vhacd.obj scale=0.001 0.001 0.001
Joints:
- joint left_finger_joint: limit lower=-0.86 upper=0 effort=20 velocity=0.2 -> lower=-0.86 upper=0 effort=200 velocity=0.2
- joint palm_left_inner_joint: limit lower=0 upper=0.86 effort=20 velocity=0.2 -> lower=0 upper=0.86 effort=200 velocity=0.2
- joint palm_left_outer_joint: limit lower=0 upper=0.86 effort=20 velocity=0.2 -> lower=0 upper=0.86 effort=200 velocity=0.2
- joint palm_right_inner_joint: limit lower=-0.86 upper=0 effort=20 velocity=0.2 -> lower=-0.86 upper=0 effort=200 velocity=0.2
- joint palm_right_outer_joint: limit lower=-0.86 upper=0 effort=20 velocity=0.2 -> lower=-0.86 upper=0 effort=200 velocity=0.2
- joint right_finger_joint: limit lower=0 upper=0.86 effort=20 velocity=0.2 -> lower=0 upper=0.86 effort=200 velocity=0.2

Commit message: uncommented visual shapes

File: burg_toolkit/gripper_module/assets/gripper/rg2/model.urdf (robot description, URDF)
Before this commit: robot rg2, 7 links, 6 joints
Links:
- link left_finger: geometry collision mesh filename=meshes/left_finger_vhacd.obj scale=0.001 0.001 0.001; visual mesh filename=meshes/left_finger_vhacd.obj scale=0.001 0.001 0.001
- link left_outer: geometry collision mesh filename=meshes/left_outer_vhacd.obj scale=0.001 0.001 0.001; visual mesh filename=meshes/left_outer_vhacd.obj scale=0.001 0.001 0.001

Commit message: increased forces for rg2, still does not hold on to grasped object

File: burg_toolkit/gripper_module/assets/gripper/rg2/model.urdf (robot description, URDF)
Before this commit: robot rg2, 7 links, 6 joints
Joints:
- joint left_finger_joint: limit lower=-0.86 upper=0 effort=200 velocity=0.2 -> lower=-0.86 upper=0 effort=1000 velocity=0.2
- joint palm_left_inner_joint: limit lower=0 upper=0.86 effort=200 velocity=0.2 -> lower=0 upper=0.86 effort=1000 velocity=0.2
- joint palm_left_outer_joint: limit lower=0 upper=0.86 effort=200 velocity=0.2 -> lower=0 upper=0.86 effort=1000 velocity=0.2
- joint palm_right_inner_joint: limit lower=-0.86 upper=0 effort=200 velocity=0.2 -> lower=-0.86 upper=0 effort=1000 velocity=0.2
- joint palm_right_outer_joint: limit lower=-0.86 upper=0 effort=200 velocity=0.2 -> lower=-0.86 upper=0 effort=1000 velocity=0.2
- joint right_finger_joint: limit lower=0 upper=0.86 effort=200 velocity=0.2 -> lower=0 upper=0.86 effort=1000 velocity=0.2
