Commit message: vhacd of meshes

File: burg_toolkit/gripper_module/assets/gripper/barrett_hand_2f/model.urdf (robot description, URDF)
Before this commit: robot bhand, 7 links, 6 joints
Links:
- link bh_base_link: geometry collision mesh filename=./meshes/palm_282.dae_vhacd.obj; visual mesh filename=./meshes/palm_282.dae_vhacd.obj
- link bh_finger_11_link: geometry collision mesh filename=./meshes/knuckle.dae_vhacd.obj; visual mesh filename=./meshes/knuckle.dae_vhacd.obj
- link bh_finger_12_link: geometry collision mesh filename=./meshes/finger.dae_vhacd.obj; visual mesh filename=./meshes/finger.dae_vhacd.obj
- link bh_finger_13_link: geometry collision mesh filename=./meshes/finger_tip.dae_vhacd.obj; visual mesh filename=./meshes/finger_tip.dae_vhacd.obj
- link bh_finger_21_link: geometry collision mesh filename=./meshes/knuckle.dae_vhacd.obj; visual mesh filename=./meshes/knuckle.dae_vhacd.obj
- link bh_finger_22_link: geometry collision mesh filename=./meshes/finger.dae_vhacd.obj; visual mesh filename=./meshes/finger.dae_vhacd.obj
- link bh_finger_23_link: geometry collision mesh filename=./meshes/finger_tip.dae_vhacd.obj; visual mesh filename=./meshes/finger_tip.dae_vhacd.obj
