Commit message: removed two fixed joints from urdf, so gripper can be moved

File: burg_toolkit/gripper_module/assets/gripper/ezgripper/model.urdf (robot description, URDF)
Before this commit: robot ezgripper_stand_alone, 7 links, 6 joints
Links:
- removed link base_link
- removed link world
Joints:
- removed joint fixed
- removed joint left_ezgripper_connect

Commit message: using vhacd meshes

File: burg_toolkit/gripper_module/assets/gripper/ezgripper/model.urdf (robot description, URDF)
Before this commit: robot ezgripper_stand_alone, 5 links, 4 joints
Links:
- link left_ezgripper_finger_L1_1: geometry collision mesh filename=meshes/SAKE_Finger_L1_Gen2_vhacd.obj
- link left_ezgripper_finger_L1_2: geometry collision mesh filename=meshes/SAKE_Finger_L1_Gen2_vhacd.obj; visual mesh filename=meshes/SAKE_Finger_L1_Gen2_vhacd.obj
- link left_ezgripper_finger_L2_1: geometry collision mesh filename=meshes/SAKE_Finger_L2_Gen2_vhacd.obj
- link left_ezgripper_finger_L2_2: geometry collision mesh filename=meshes/SAKE_Finger_L2_Gen2_vhacd.obj; visual mesh filename=meshes/SAKE_Finger_L2_Gen2_vhacd.obj
- link left_ezgripper_palm_link: geometry collision mesh filename=meshes/SAKE_Palm_Dual_Gen2_vhacd.obj

Commit message: uncomment visual shapes

File: burg_toolkit/gripper_module/assets/gripper/ezgripper/model.urdf (robot description, URDF)
Before this commit: robot ezgripper_stand_alone, 5 links, 4 joints
Links:
- link left_ezgripper_finger_L1_1: geometry collision mesh filename=meshes/SAKE_Finger_L1_Gen2_vhacd.obj; visual mesh filename=meshes/SAKE_Finger_L1_Gen2_vhacd.obj
- link left_ezgripper_finger_L2_1: geometry collision mesh filename=meshes/SAKE_Finger_L2_Gen2_vhacd.obj; visual mesh filename=meshes/SAKE_Finger_L2_Gen2_vhacd.obj
- link left_ezgripper_palm_link: geometry collision mesh filename=meshes/SAKE_Palm_Dual_Gen2_vhacd.obj; visual mesh filename=meshes/SAKE_Palm_Dual_Gen2_vhacd.obj
