Commit message: stl to vhacd

File: burg_toolkit/gripper_module/assets/gripper/franka/model.urdf (robot description, URDF)
Before this commit: robot panda, 3 links, 2 joints
Links:
- link panda_hand: geometry collision mesh filename=meshes/hand_vhacd.obj; visual mesh filename=meshes/hand_vhacd.obj
- link panda_leftfinger: geometry collision mesh filename=meshes/finger_vhacd.obj; visual mesh filename=meshes/finger_vhacd.obj
- link panda_rightfinger: geometry collision mesh filename=meshes/finger_vhacd.obj; visual mesh filename=meshes/finger_vhacd.obj
