Commit message: stl to vhacd

File: burg_toolkit/gripper_module/assets/gripper/wsg_50/model.urdf (robot description, URDF)
Before this commit: robot wsg_50, 5 links, 4 joints
Links:
- link base_link: geometry collision mesh filename=./meshes/WSG50_110_vhacd.obj scale=1 1 1; visual mesh filename=./meshes/WSG50_110_vhacd.obj scale=1 1 1
- link finger_left: geometry collision mesh filename=./meshes/WSG-FMF_vhacd.obj scale=0.001 0.001 0.001; visual mesh filename=./meshes/WSG-FMF_vhacd.obj scale=0.001 0.001 0.001
- link finger_right: geometry collision mesh filename=./meshes/WSG-FMF_vhacd.obj scale=0.001 0.001 0.001; visual mesh filename=./meshes/WSG-FMF_vhacd.obj scale=0.001 0.001 0.001
- link gripper_left: geometry collision mesh filename=./meshes/GUIDE_WSG50_110_vhacd.obj scale=0.001 0.001 0.001; visual mesh filename=./meshes/GUIDE_WSG50_110_vhacd.obj scale=0.001 0.001 0.001
- link gripper_right: geometry collision mesh filename=./meshes/GUIDE_WSG50_110_vhacd.obj scale=0.001 0.001 0.001; visual mesh filename=./meshes/GUIDE_WSG50_110_vhacd.obj scale=0.001 0.001 0.001
