Commit message: adjusted visual shapes of pads to fit collision shapes

File: burg_toolkit/gripper_module/assets/gripper/robotiq_2f_140/model.urdf (robot description, URDF)
Before this commit: robot robotiq_arg2f_140_model, 11 links, 10 joints
Links:
- link left_inner_finger_pad: geometry collision box size=0.03 0.07 0.0075; visual box size=0.03 0.07 0.0075
- link right_inner_finger_pad: geometry collision box size=0.03 0.07 0.0075; visual box size=0.03 0.07 0.0075

Commit message: stl to vhacd

File: burg_toolkit/gripper_module/assets/gripper/robotiq_2f_140/model.urdf (robot description, URDF)
Before this commit: robot robotiq_arg2f_140_model, 11 links, 10 joints
Links:
- link left_inner_finger: geometry visual mesh filename=./meshes/robotiq_arg2f_140_inner_finger_vhacd.obj
- link left_inner_knuckle: geometry collision mesh filename=./meshes/robotiq_arg2f_140_inner_knuckle_vhacd.obj; visual mesh filename=./meshes/robotiq_arg2f_140_inner_knuckle_vhacd.obj
- link left_outer_finger: geometry collision mesh filename=./meshes/robotiq_arg2f_140_outer_finger_vhacd.obj; visual mesh filename=./meshes/robotiq_arg2f_140_outer_finger_vhacd.obj
- link left_outer_knuckle: geometry collision mesh filename=./meshes/robotiq_arg2f_140_outer_knuckle_vhacd.obj; visual mesh filename=./meshes/robotiq_arg2f_140_outer_knuckle_vhacd.obj
- link right_inner_finger: geometry visual mesh filename=./meshes/robotiq_arg2f_140_inner_finger_vhacd.obj
- link right_inner_knuckle: geometry collision mesh filename=./meshes/robotiq_arg2f_140_inner_knuckle_vhacd.obj; visual mesh filename=./meshes/robotiq_arg2f_140_inner_knuckle_vhacd.obj
- link right_outer_finger: geometry collision mesh filename=./meshes/robotiq_arg2f_140_outer_finger_vhacd.obj; visual mesh filename=./meshes/robotiq_arg2f_140_outer_finger_vhacd.obj
- link right_outer_knuckle: geometry collision mesh filename=./meshes/robotiq_arg2f_140_outer_knuckle_vhacd.obj; visual mesh filename=./meshes/robotiq_arg2f_140_outer_knuckle_vhacd.obj
- link robotiq_arg2f_base_link: geometry collision mesh filename=./meshes/robotiq_arg2f_base_link_vhacd.obj; visual mesh filename=./meshes/robotiq_arg2f_base_link_vhacd.obj
