Commit message: greater joint range, increased max velocity

File: burg_toolkit/assets/dummy_xyz_robot.urdf (robot description, URDF)
Before this commit: robot dummy_xyz_robot, 4 links, 3 joints
Joints:
- joint center_x: limit lower=-0.5 upper=0.5 effort=1000.0 velocity=0.2 -> lower=-1 upper=1 effort=1000.0 velocity=0.5
- joint center_y: limit lower=-0.5 upper=0.5 effort=1000.0 velocity=0.2 -> lower=-1 upper=1 effort=1000.0 velocity=0.5
- joint center_z: limit lower=-0.5 upper=0.5 effort=1000.0 velocity=0.2 -> lower=-1 upper=1 effort=1000.0 velocity=0.5
